Commit message: second commit

File: xacro/gazebo/stereo_camera.xacro (robot description, xacro)
@@ -22,5 +22,6 @@
         </camera>
         <camera name="right">
-          <pose>0 -0.1 0 0.00410 -0.00417 0.01106 </pose>
+          <pose>0 -0.3 0 0.00410 -0.00417 0.01106 </pose>
+          <!-- <pose>0 -0.2 0 0 0 0 </pose> -->
           <horizontal_fov>1.3962634</horizontal_fov>
           <image>
@@ -46,5 +47,5 @@
           <cameraInfoTopicName>camera_info</cameraInfoTopicName>
           <frameName>camera</frameName>
-          <hackBaseline>0.1</hackBaseline>
+          <hackBaseline>0.3</hackBaseline>
           <distortionK1>-0.28340811</distortionK1>
           <distortionK2>0.07395907</distortionK2>
@@ -52,4 +53,9 @@
           <distortionT1>0.00019359</distortionT1>
           <distortionT2>1.76187114e-05</distortionT2>
+          <!-- <distortionK1>0.0</distortionK1>
+          <distortionK2>0.0</distortionK2>
+          <distortionK3>0.0</distortionK3>
+          <distortionT1>0.0</distortionT1>
+          <distortionT2>0.0</distortionT2> -->
         </plugin>
       </sensor>

File: xacro/my_base.xacro (robot description, xacro)
@@ -10,5 +10,5 @@
     <!-- 封装变量、常量 -->
     <!-- PI 值设置精度需要高一些，否则后续车轮翻转量计算时，可能会出现肉眼不能察觉的车轮倾斜，从而导致模型抖动 -->
-    <xacro:property name="PI" value="3.1415926"/>
+    <xacro:property name="PI" value="3.14159265358979323846"/>
     <!-- 宏:黑色设置 -->
     <material name="black">
@@ -17,5 +17,5 @@
     <!-- 底盘属性 -->
     <xacro:property name="base_footprint_radius" value="0.001" /> <!-- base_footprint 半径  -->
-    <xacro:property name="base_link_radius" value="0.1" /> <!-- base_link 半径 -->
+    <xacro:property name="base_link_radius" value="0.15" /> <!-- base_link 半径 -->
     <xacro:property name="base_link_length" value="0.08" /> <!-- base_link 长 -->
     <xacro:property name="earth_space" value="0.015" /> <!-- 离地间距 -->
@@ -57,7 +57,7 @@
     <!-- 驱动轮 -->
     <!-- 驱动轮属性 -->
-    <xacro:property name="wheel_radius" value="0.0325" /><!-- 半径 -->
-    <xacro:property name="wheel_length" value="0.015" /><!-- 宽度 -->
-    <xacro:property name="wheel_m" value="0.05" /> <!-- 质量  -->
+    <xacro:property name="wheel_radius" value="0.05" /><!-- 半径 -->
+    <xacro:property name="wheel_length" value="0.03" /><!-- 宽度 -->
+    <xacro:property name="wheel_m" value="0.5" /> <!-- 质量  -->
     <!-- 驱动轮宏实现 -->
     <xacro:macro name="add_wheels" params="name flag">
